Commit message: Add sensors peripherals and recording updates

File: src/robot_arm3/urdf/robot_arm3_control_05.urdf.xacro (robot description, xacro)
@@ -9,8 +9,13 @@
     name="controller_config"
     default="$(find robot_arm3)/config/ros2_controllers_05.yaml" />
+  <!-- Tool offsets are relative to the calibrated C4G flange frame. -->
+  <xacro:arg name="tcp_xyz" default="0 0 0" />
+  <xacro:arg name="tcp_rpy" default="0 0 0" />
   <link
     name="world" />
-  <joint
-    name="world_to_base_link"
+  <link
+    name="c4g_base" />
+  <joint
+    name="world_to_c4g_base"
     type="fixed">
     <origin
@@ -19,4 +24,15 @@
     <parent
       link="world" />
+    <child
+      link="c4g_base" />
+  </joint>
+  <joint
+    name="c4g_base_to_base_link"
+    type="fixed">
+    <origin
+      xyz="0 0 0"
+      rpy="0 0 3.141592653589793" />
+    <parent
+      link="c4g_base" />
     <child
       link="base_link" />
@@ -412,4 +428,17 @@
       effort="2000"
       velocity="1" />
+  </joint>
+  <!-- Link_6 uses the exported CAD frame. This fixed frame matches C4G tool0. -->
+  <link name="c4g_flange_link" />
+  <joint name="link6_to_c4g_flange" type="fixed">
+    <origin xyz="0 0 -0.023506" rpy="0 3.141592653589793 0" />
+    <parent link="Link_6" />
+    <child link="c4g_flange_link" />
+  </joint>
+  <link name="tcp_link" />
+  <joint name="flange_to_tcp" type="fixed">
+    <origin xyz="$(arg tcp_xyz)" rpy="$(arg tcp_rpy)" />
+    <parent link="c4g_flange_link" />
+    <child link="tcp_link" />
   </joint>
   <link

File: src/robot_arm3/urdf/robot_arm3_moveit.urdf.xacro (robot description, xacro)
@@ -6,4 +6,13 @@
   name="robot_arm3"
   xmlns:xacro="http://www.ros.org/wiki/xacro">
+  <!-- Configure the static tool before launch. xyz is metres; rpy is radians. -->
+  <xacro:arg name="tcp_xyz" default="0 0 0" />
+  <xacro:arg name="tcp_rpy" default="0 0 0" />
+  <link name="c4g_base" />
+  <joint name="c4g_base_to_base_link" type="fixed">
+    <origin xyz="0 0 0" rpy="0 0 3.141592653589793" />
+    <parent link="c4g_base" />
+    <child link="base_link" />
+  </joint>
   <link
     name="base_link">
@@ -397,4 +406,17 @@
       velocity="1" />
   </joint>
+  <!-- Link_6 uses the exported CAD frame. This fixed frame matches C4G tool0. -->
+  <link name="c4g_flange_link" />
+  <joint name="link6_to_c4g_flange" type="fixed">
+    <origin xyz="0 0 -0.023506" rpy="0 3.141592653589793 0" />
+    <parent link="Link_6" />
+    <child link="c4g_flange_link" />
+  </joint>
+  <link name="tcp_link" />
+  <joint name="flange_to_tcp" type="fixed">
+    <origin xyz="$(arg tcp_xyz)" rpy="$(arg tcp_rpy)" />
+    <parent link="c4g_flange_link" />
+    <child link="tcp_link" />
+  </joint>
   <link
     name="Link_7">
