Commit message: Update project files for submission

File: src/robot_arm3/urdf/robot_arm3_control_05.urdf.xacro (robot description, xacro)
@@ -12,4 +12,7 @@
   <xacro:arg name="tcp_xyz" default="0 0 0" />
   <xacro:arg name="tcp_rpy" default="0 0 0" />
+  <xacro:arg name="fixture_rod_length" default="0.20" />
+  <xacro:arg name="fixture_rod_radius" default="0.013" />
+  <xacro:include filename="$(find robot_arm3)/urdf/rod_fixture.xacro" />
   <link
     name="world" />
@@ -20,5 +23,5 @@
     type="fixed">
     <origin
-      xyz="0 0 0"
+      xyz="0 0 0.08"
       rpy="0 0 0" />
     <parent
@@ -26,4 +29,32 @@
     <child
       link="c4g_base" />
+  </joint>
+  <!--
+    The physical robot is mounted on an 80 mm pedestal.  c4g_base remains
+    the C4G programming origin on the pedestal's top face; the pedestal
+    therefore extends downward from this frame to the Gazebo ground plane.
+    Its footprint encloses the base-link mesh bounding box with 200 mm
+    clearance on every side.
+  -->
+  <link name="pedestal_link">
+    <visual>
+      <origin xyz="-0.18 0.068663731 -0.04" rpy="0 0 0" />
+      <geometry>
+        <box size="1.75 1.4243275 0.08" />
+      </geometry>
+      <material name="pedestal_gray">
+        <color rgba="0.24 0.24 0.27 1" />
+      </material>
+    </visual>
+    <collision>
+      <origin xyz="-0.18 0.068663731 -0.04" rpy="0 0 0" />
+      <geometry>
+        <box size="1.75 1.4243275 0.08" />
+      </geometry>
+    </collision>
+  </link>
+  <joint name="c4g_base_to_pedestal" type="fixed">
+    <parent link="c4g_base" />
+    <child link="pedestal_link" />
   </joint>
   <joint
@@ -436,10 +467,9 @@
     <child link="c4g_flange_link" />
   </joint>
-  <link name="tcp_link" />
-  <joint name="flange_to_tcp" type="fixed">
-    <origin xyz="$(arg tcp_xyz)" rpy="$(arg tcp_rpy)" />
-    <parent link="c4g_flange_link" />
-    <child link="tcp_link" />
-  </joint>
+  <xacro:rod_fixture
+    flange_xyz="$(arg tcp_xyz)"
+    flange_rpy="$(arg tcp_rpy)"
+    rod_length="$(arg fixture_rod_length)"
+    rod_radius="$(arg fixture_rod_radius)" />
   <link
     name="Link_7">

File: src/robot_arm3/urdf/robot_arm3_moveit.urdf.xacro (robot description, xacro)
@@ -9,5 +9,30 @@
   <xacro:arg name="tcp_xyz" default="0 0 0" />
   <xacro:arg name="tcp_rpy" default="0 0 0" />
+  <xacro:arg name="fixture_rod_length" default="0.20" />
+  <xacro:arg name="fixture_rod_radius" default="0.013" />
+  <xacro:include filename="$(find robot_arm3)/urdf/rod_fixture.xacro" />
   <link name="c4g_base" />
+  <!-- 80 mm support below c4g_base; dimensions clear the base mesh by 200 mm. -->
+  <link name="pedestal_link">
+    <visual>
+      <origin xyz="-0.18 0.068663731 -0.04" rpy="0 0 0" />
+      <geometry>
+        <box size="1.75 1.4243275 0.08" />
+      </geometry>
+      <material name="pedestal_gray">
+        <color rgba="0.24 0.24 0.27 1" />
+      </material>
+    </visual>
+    <collision>
+      <origin xyz="-0.18 0.068663731 -0.04" rpy="0 0 0" />
+      <geometry>
+        <box size="1.75 1.4243275 0.08" />
+      </geometry>
+    </collision>
+  </link>
+  <joint name="c4g_base_to_pedestal" type="fixed">
+    <parent link="c4g_base" />
+    <child link="pedestal_link" />
+  </joint>
   <joint name="c4g_base_to_base_link" type="fixed">
     <origin xyz="0 0 0" rpy="0 0 3.141592653589793" />
@@ -413,10 +438,9 @@
     <child link="c4g_flange_link" />
   </joint>
-  <link name="tcp_link" />
-  <joint name="flange_to_tcp" type="fixed">
-    <origin xyz="$(arg tcp_xyz)" rpy="$(arg tcp_rpy)" />
-    <parent link="c4g_flange_link" />
-    <child link="tcp_link" />
-  </joint>
+  <xacro:rod_fixture
+    flange_xyz="$(arg tcp_xyz)"
+    flange_rpy="$(arg tcp_rpy)"
+    rod_length="$(arg fixture_rod_length)"
+    rod_radius="$(arg fixture_rod_radius)" />
   <link
     name="Link_7">
